File: rev_a/bus_beaglebone.kicad_pcb (KiCad board)
At the start: 2 copper layers, 100 x 50 mm, 39 parts, among them J1 TERMINATE_JUMPER, J2 LED_JUMPER, Q1 FQP47P06, SW1 MJTP1243, U1 74HCT08, U2 MCP2562, U3 ATMEGA324_DIP40, X1 16MHz, X2 OSHW_LOGO

Commit message: Finnished doing clone of bus_raspberry_pi.
Parts:
- C1, C2, C3, C4, C5, C6, C7, C8: footprint Bus_Raspberry_Pi_Rev_A:Capacitor3MMDiscRM2.5 -> Bus_BeagleBone_Rev_A:Capacitor3MMDiscRM2.5
- D1: footprint Bus_Raspberry_Pi_Rev_A:Diode_DO-41_SOD81_Horizontal_RM10 -> Bus_BeagleBone_Rev_A:Diode_DO-41_SOD81_Horizontal_RM10
- D2: footprint Bus_Raspberry_Pi_Rev_A:T1_LED -> Bus_BeagleBone_Rev_A:T1_LED
- H1, H2, H3, H4: footprint Bus_Raspberry_Pi_Rev_A:MountingHole_3mm -> Bus_BeagleBone_Rev_A:MountingHole_3mm
- J1: footprint Bus_Raspberry_Pi_Rev_A:Pin_Header_Straight_1x03 -> Bus_BeagleBone_Rev_A:Pin_Header_Straight_1x03
- J2: footprint Bus_Raspberry_Pi_Rev_A:Pin_Header_Straight_2x02 -> Bus_BeagleBone_Rev_A:Pin_Header_Straight_2x02
- N1, N2: footprint Bus_Raspberry_Pi_Rev_A:5MM_TERMINAL_BLOCK_2_POS -> Bus_BeagleBone_Rev_A:5MM_TERMINAL_BLOCK_2_POS
- N10: footprint Bus_Raspberry_Pi_Rev_A:Pin_Header_Straight_2x20 -> Bus_BeagleBone_Rev_A:Pin_Header_Straight_2x20
- N3, N9: footprint Bus_Raspberry_Pi_Rev_A:Pin_Header_Straight_2x05_Shrouded -> Bus_BeagleBone_Rev_A:Pin_Header_Straight_2x05_Shrouded
- N4, N5: footprint Bus_Raspberry_Pi_Rev_A:Pin_Header_Straight_1x06 -> Bus_BeagleBone_Rev_A:Pin_Header_Straight_1x06
- N6: footprint Bus_Raspberry_Pi_Rev_A:OKI_DC_TO_DC_CONNECTOR -> Bus_BeagleBone_Rev_A:OKI_DC_TO_DC_CONNECTOR
- N7: footprint Bus_Raspberry_Pi_Rev_A:Pin_Header_Straight_2x03 -> Bus_BeagleBone_Rev_A:Pin_Header_Straight_2x03
- N8: footprint Bus_Raspberry_Pi_Rev_A:Pin_Header_Straight_1x04 -> Bus_BeagleBone_Rev_A:Pin_Header_Straight_1x04
- Q1: footprint Bus_Raspberry_Pi_Rev_A:TO-220_FET-GDS_Horizontal_LargePads -> Bus_BeagleBone_Rev_A:TO-220_FET-GDS_Horizontal_LargePads
- R1, R2: footprint Bus_Raspberry_Pi_Rev_A:Pin_Header_Straight_1x08 -> Bus_BeagleBone_Rev_A:Pin_Header_Straight_1x08
- R3, R4, R5, R6: footprint Bus_Raspberry_Pi_Rev_A:Resistor_Horizontal__400 -> Bus_BeagleBone_Rev_A:Resistor_Horizontal__400
- SW1: footprint Bus_Raspberry_Pi_Rev_A:Button_6.5MM -> Bus_BeagleBone_Rev_A:Button_6.5MM
- U1: footprint Bus_Raspberry_Pi_Rev_A:DIP-14__300 -> Bus_BeagleBone_Rev_A:DIP-14__300
- U2: footprint Bus_Raspberry_Pi_Rev_A:DIP-8__300 -> Bus_BeagleBone_Rev_A:DIP-8__300
- U3: footprint Bus_Raspberry_Pi_Rev_A:DIP-40__600 -> Bus_BeagleBone_Rev_A:DIP-40__600
- X1: footprint Bus_Raspberry_Pi_Rev_A:Crystal_HC49-U_Vertical -> Bus_BeagleBone_Rev_A:Crystal_HC49-U_Vertical
- X2: footprint Bus_Raspberry_Pi_Rev_A:OSHW_LOGO_200mil -> Bus_BeagleBone_Rev_A:OSHW_LOGO_250mil
- moved X2 0.70 mm to (134.1, 124.6)

Commit message: Updated again.
Parts:
- N10: value RASPI_CONNECTOR_40 -> BBB_P9_HEADER; footprint Bus_BeagleBone_Rev_A:Pin_Header_Straight_2x20 -> Bus_BeagleBone_Rev_A:Pin_Header_Straight_2x16
- moved N10 5.72 mm to (121.9, 104.8)
Connections:
- N10 pad 1: Net-(N10-Pad1) -> GND
- N10 pad 14: GND -> Net-(N10-Pad14)
- N10 pad 2: +5V -> GND
- N10 pad 20: GND -> Net-(N10-Pad20)
- N10 pad 25: GND -> Net-(N10-Pad25)
- N10 pad 30: GND -> Net-(N10-Pad30)
- N10 pad 4: +5V -> Net-(N10-Pad4)
- N10 pad 5: Net-(N10-Pad5) -> +5V
- N10 pad 6: Net-(N10-Pad6) -> +5V
- N10 pad 9: GND -> Net-(N10-Pad9)
- N5 pad 5: Net-(N10-Pad8) -> Net-(N10-Pad21)
- N8 pad 2: Net-(N10-Pad8) -> Net-(N10-Pad21)
- N8 pad 3: Net-(N10-Pad10) -> Net-(N10-Pad22)
- N8 pad 4: Net-(N10-Pad26) -> Net-(N10-Pad31)
- R1 pad 6: Net-(N10-Pad10) -> Net-(N10-Pad22)
- R1 pad 7: Net-(N10-Pad26) -> Net-(N10-Pad31)
- R1 pad 8: Net-(N10-Pad8) -> Net-(N10-Pad21)
- R2 pad 6: Net-(N10-Pad10) -> Net-(N10-Pad22)
- R2 pad 7: Net-(N10-Pad26) -> Net-(N10-Pad31)
- R2 pad 8: Net-(N10-Pad8) -> Net-(N10-Pad21)
- U1 pad 12: Net-(N10-Pad26) -> Net-(N10-Pad31)
- U1 pad 5: Net-(N10-Pad8) -> Net-(N10-Pad21)
Routing:
- net Net-(N10-Pad8): track 136.6 -> 0.00 mm, vias 3 -> 0
- net Net-(N10-Pad21): track 0.00 -> 111.6 mm, vias 0 -> 2
- net Net-(N10-Pad26): track 85.2 -> 0.00 mm, vias 3 -> 0
- net Net-(N10-Pad10): track 80.6 -> 0.00 mm, vias 1 -> 0
- net Net-(N10-Pad31): track 0.00 -> 76.8 mm, vias 0 -> 3
- net Net-(N10-Pad22): track 0.00 -> 66.9 mm, vias 0 -> 1
- net GND: track 174.9 -> 133.0 mm, vias 1 -> 0
- net +5V: track 240.9 -> 229.8 mm, vias 3 -> 2
Other:
- board text added: "BUS BEAGLEBONE REV A. 10AUG2014 (c) 2014 GRAMLICH"
- board text removed: "BUS RASPBERRY PI REV A. 10AUG2014 (c) 2014 GRAMLICH"
