File: rev_b/bus_beaglebone.kicad_pcb (KiCad board)
At the start: 2 copper layers, 100 x 50 mm, 39 parts, among them J1 TERMINATE_JUMPER, J2 LED_JUMPER, Q1 FQP47P06, SW1 MJTP1243, U1 74HCT08, U2 MCP2562, U3 ATMEGA324_DIP40, X1 16MHz, X2 OSHW_LOGO

Commit message: Got Rev. B in pretty good shape.
Parts:
- added R7: 22K, bus_beaglebone:Resistor_Horizontal__400, F.Cu at (161.3, 109.9)
- added R8: 33K, bus_beaglebone:Pin_Header_Straight_1x05, F.Cu at (175.9, 116.2)
- C1, C2, C3, C4, C5, C7: footprint Bus_BeagleBone_Rev_A:Capacitor3MMDiscRM2.5 -> bus_beaglebone:Capacitor3MMDiscRM2.5
- C6, C8: value .1uF -> 1uF; footprint Bus_BeagleBone_Rev_A:Capacitor3MMDiscRM2.5 -> bus_beaglebone:Capacitor3MMDiscRM2.5
- D1: footprint Bus_BeagleBone_Rev_A:Diode_DO-41_SOD81_Horizontal_RM10 -> bus_beaglebone:Diode_DO-41_SOD81_Horizontal_RM10
- D2: footprint Bus_BeagleBone_Rev_A:T1_LED -> bus_beaglebone:T1_LED
- H1, H2, H3, H4: footprint Bus_BeagleBone_Rev_A:MountingHole_3mm -> bus_beaglebone:MountingHole_3mm
- J1: footprint Bus_BeagleBone_Rev_A:Pin_Header_Straight_1x03 -> bus_beaglebone:Pin_Header_Straight_1x03
- J2: footprint Bus_BeagleBone_Rev_A:Pin_Header_Straight_2x02 -> bus_beaglebone:Pin_Header_Straight_2x02
- N1, N2: footprint Bus_BeagleBone_Rev_A:5MM_TERMINAL_BLOCK_2_POS -> bus_beaglebone:5MM_TERMINAL_BLOCK_2_POS
- N10: footprint Bus_BeagleBone_Rev_A:Pin_Header_Straight_2x16 -> bus_beaglebone:Pin_Header_Straight_2x23
- N3, N9: footprint Bus_BeagleBone_Rev_A:Pin_Header_Straight_2x05_Shrouded -> bus_beaglebone:Pin_Header_Straight_2x05_Shrouded
- N4, N5: footprint Bus_BeagleBone_Rev_A:Pin_Header_Straight_1x06 -> bus_beaglebone:Pin_Header_Straight_1x06
- N6: footprint Bus_BeagleBone_Rev_A:OKI_DC_TO_DC_CONNECTOR -> bus_beaglebone:OKI_DC_TO_DC_CONNECTOR
- N7: footprint Bus_BeagleBone_Rev_A:Pin_Header_Straight_2x03 -> bus_beaglebone:Pin_Header_Straight_2x03
- N8: footprint Bus_BeagleBone_Rev_A:Pin_Header_Straight_1x04 -> bus_beaglebone:Pin_Header_Straight_1x04
- Q1: footprint Bus_BeagleBone_Rev_A:TO-220_FET-GDS_Horizontal_LargePads -> bus_beaglebone:TO-220_FET-GDS_Horizontal_LargePads
- R1: footprint Bus_BeagleBone_Rev_A:Pin_Header_Straight_1x08 -> bus_beaglebone:Pin_Header_Straight_1x05
- R2: value 33K -> 22K; footprint Bus_BeagleBone_Rev_A:Pin_Header_Straight_1x08 -> bus_beaglebone:Resistor_Horizontal__400
- R3, R4, R5, R6: footprint Bus_BeagleBone_Rev_A:Resistor_Horizontal__400 -> bus_beaglebone:Resistor_Horizontal__400
- SW1: footprint Bus_BeagleBone_Rev_A:Button_6.5MM -> bus_beaglebone:Button_6.5MM
- U1: footprint Bus_BeagleBone_Rev_A:DIP-14__300 -> bus_beaglebone:DIP-14__300
- U2: footprint Bus_BeagleBone_Rev_A:DIP-8__300 -> bus_beaglebone:DIP-8__300
- U3: footprint Bus_BeagleBone_Rev_A:DIP-40__600 -> bus_beaglebone:DIP-40__600
- X1: footprint Bus_BeagleBone_Rev_A:Crystal_HC49-U_Vertical -> bus_beaglebone:Crystal_HC49-U_Vertical
- X2: footprint Bus_BeagleBone_Rev_A:OSHW_LOGO_250mil -> bus_beaglebone:OSHW_LOGO_250mil
- moved X2 61.5 mm to (194.3, 111.8)
- moved R2 40.6 mm to (136.5, 116.8), turned to 180 degrees
- moved R4 36.7 mm to (121.3, 123.2), turned to 270 degrees
- moved D1 36.3 mm to (123.8, 114.9), turned to 180 degrees
- moved SW1 34.1 mm to (188.0, 144.8), turned to 90 degrees
- moved C6 14.3 mm to (151.1, 109.9), turned to 180 degrees
- moved R6 10.3 mm to (119.4, 111.8)
- moved R5 9.71 mm to (119.4, 108.6)
- moved D2 9.71 mm to (109.9, 110.5), turned to 180 degrees
- moved N10 8.91 mm to (130.8, 104.1)
- moved N4 6.98 mm to (138.4, 109.9)
- moved N8 5.08 mm to (135.9, 113.7)
- moved C8 4.26 mm to (162.6, 105.4), turned to 90 degrees
- moved J2 4.02 mm to (113.7, 116.2), turned to 180 degrees
- moved C1 2.54 mm to (149.9, 143.5), turned to 90 degrees
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Connections:
- J1 pad 3: Net-(J1-Pad3) -> (no net)
- N10 pad 10: Net-(N10-Pad10) -> (no net)
- N10 pad 11: Net-(N10-Pad11) -> (no net)
- N10 pad 12: Net-(N10-Pad12) -> (no net)
- N10 pad 13: Net-(N10-Pad13) -> (no net)
- N10 pad 14: Net-(N10-Pad14) -> (no net)
- N10 pad 15: Net-(N10-Pad15) -> (no net)
- N10 pad 16: Net-(N10-Pad16) -> (no net)
- N10 pad 17: Net-(N10-Pad17) -> (no net)
- N10 pad 18: Net-(N10-Pad18) -> (no net)
- N10 pad 19: Net-(N10-Pad19) -> (no net)
- N10 pad 20: Net-(N10-Pad20) -> (no net)
- N10 pad 23: Net-(N10-Pad23) -> (no net)
- N10 pad 24: Net-(N10-Pad24) -> (no net)
- N10 pad 25: Net-(N10-Pad25) -> (no net)
- N10 pad 26: Net-(N10-Pad26) -> (no net)
- N10 pad 27: Net-(N10-Pad27) -> (no net)
- N10 pad 28: Net-(N10-Pad28) -> (no net)
- N10 pad 29: Net-(N10-Pad29) -> (no net)
- N10 pad 3: Net-(N10-Pad3) -> (no net)
- N10 pad 30: Net-(N10-Pad30) -> (no net)
- N10 pad 32: Net-(N10-Pad32) -> (no net)
- N10 pad 4: Net-(N10-Pad4) -> (no net)
- N10 pad 7: Net-(N10-Pad7) -> (no net)
- N10 pad 8: Net-(N10-Pad8) -> (no net)
- N10 pad 9: Net-(N10-Pad9) -> (no net)
- N3 pad 1: Net-(N3-Pad1) -> (no net)
- N3 pad 10: Net-(N3-Pad10) -> (no net)
- N3 pad 2: Net-(N3-Pad2) -> (no net)
- N3 pad 7: Net-(N3-Pad7) -> (no net)
- N3 pad 8: Net-(N3-Pad8) -> (no net)
- N3 pad 9: Net-(N3-Pad9) -> (no net)
- N4 pad 2: Net-(N4-Pad2) -> (no net)
- N4 pad 3: Net-(N4-Pad3) -> (no net)
- N5 pad 2: Net-(N5-Pad2) -> (no net)
- N5 pad 3: Net-(N5-Pad3) -> (no net)
- N5 pad 6: Net-(N5-Pad6) -> (no net)
- N9 pad 6: Net-(C8-Pad2) -> /SCK
- N9 pad 7: Net-(N9-Pad7) -> (no net)
- N9 pad 8: Net-(N9-Pad8) -> (no net)
- R1 pad 2: Net-(N5-Pad4) -> Net-(N4-Pad6)
- R1 pad 3: Net-(N4-Pad6) -> Net-(N4-Pad4)
- R1 pad 4: Net-(N4-Pad4) -> Net-(N10-Pad31)
- R1 pad 5: Net-(N4-Pad5) -> Net-(N10-Pad21)
- R2 pad 1: GND -> Net-(N4-Pad5)
- R2 pad 2: Net-(N5-Pad4) -> /TXD0
- U1 pad 9: Net-(N4-Pad5) -> /TXD0
- U2 pad 1: /RXD1 -> /TXD1
- U2 pad 4: /TXD1 -> /RXD1
- U2 pad 8: GND -> Net-(U2-Pad8)
- U3 pad 1: Net-(U3-Pad1) -> (no net)
- U3 pad 18: Net-(U3-Pad18) -> (no net)
- U3 pad 19: Net-(U3-Pad19) -> (no net)
- U3 pad 2: Net-(U3-Pad2) -> (no net)
- U3 pad 20: Net-(U3-Pad20) -> Net-(U2-Pad8)
- U3 pad 21: Net-(U3-Pad21) -> (no net)
- U3 pad 22: Net-(U3-Pad22) -> (no net)
- U3 pad 23: Net-(U3-Pad23) -> (no net)
- U3 pad 28: Net-(U3-Pad28) -> (no net)
- U3 pad 29: Net-(U3-Pad29) -> (no net)
- U3 pad 3: Net-(U3-Pad3) -> (no net)
- U3 pad 32: Net-(U3-Pad32) -> (no net)
- U3 pad 33: Net-(U3-Pad33) -> (no net)
- U3 pad 34: Net-(U3-Pad34) -> (no net)
- U3 pad 35: Net-(U3-Pad35) -> (no net)
- U3 pad 36: Net-(U3-Pad36) -> (no net)
- U3 pad 37: Net-(U3-Pad37) -> (no net)
- U3 pad 38: Net-(U3-Pad38) -> (no net)
- U3 pad 39: Net-(U3-Pad39) -> (no net)
- U3 pad 4: Net-(U3-Pad4) -> (no net)
- U3 pad 40: Net-(U3-Pad40) -> (no net)
- U3 pad 5: Net-(U3-Pad5) -> (no net)
Routing:
- net GND: track 133.0 -> 348.7 mm, vias 0 -> 18
- net /TXD0: track 0.00 -> 97.4 mm, vias 0 -> 4
- net Net-(C8-Pad2): track 68.4 -> 18.0 mm, vias 1 -> 0
- net /SCK: track 38.9 -> 88.7 mm, vias 0 -> 1
- net /~RESET: track 91.3 -> 137.6 mm, vias 2 -> 0
- net Net-(U2-Pad8): track 0.00 -> 31.5 mm
- net Net-(R7-Pad2): track 0.00 -> 31.2 mm
- net Net-(N5-Pad4): track 90.5 -> 111.2 mm
- net Net-(N4-Pad4): track 39.5 -> 55.1 mm
- net Net-(N10-Pad31): track 76.8 -> 62.6 mm, vias 3 -> 0
- net +5V: track 229.8 -> 218.5 mm, vias 2 -> 1
- net Net-(C6-Pad1): track 15.1 -> 25.5 mm, vias 1 -> 0
- net Net-(J2-Pad1): track 13.5 -> 3.44 mm
- net Net-(N10-Pad21): track 111.6 -> 103.9 mm, vias 2 -> 0
- net Net-(N4-Pad5): track 47.5 -> 40.3 mm
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Other:
- board text added: "BUS BEAGLEBONE REV. B 4OCT2014 (c) 2014 GRAMLICH"
- board text added: "RESET"
- board text removed: "BUS BEAGLEBONE REV A. 10AUG2014 (c) 2014 GRAMLICH"
