File: rev_b/bus_beaglebone.sch (KiCad schematic (older format))
At the start: 39 parts, among them J1 TERMINATE_JUMPER, J2 LED_JUMPER, Q1 FQP47P06, SW1 MJTP1243, U1 74HCT08, U2 MCP2562, U3 ATMEGA324_DIP40, X1 16MHz, X2 OSHW_LOGO

Commit message: Got Rev. B in pretty good shape.
Parts:
- removed R1: 22Kx, symbol R_VERT_SIP8
- removed R2: 33Kx, symbol R_VERT_SIP8
- added R1: 22K, bus_beaglebone:Pin_Header_Straight_1x05, symbol R_VERT_SIP5
- added R2, R7: 22K, bus_beaglebone:Resistor_Horizontal__400, symbol R_VERT
- added R8: 33K, bus_beaglebone:Pin_Header_Straight_1x05, symbol R_VERT_SIP5_ALT
- C1, C2, C3, C4, C5, C7: footprint (none) -> bus_beaglebone:Capacitor3MMDiscRM2.5
- C6, C8: value .1uF -> 1uF; footprint (none) -> bus_beaglebone:Capacitor3MMDiscRM2.5
- D1: footprint (none) -> bus_beaglebone:Diode_DO-41_SOD81_Horizontal_RM10
- D2: footprint (none) -> bus_beaglebone:T1_LED
- H1, H2, H3, H4: footprint (none) -> bus_beaglebone:MountingHole_3mm
- J1: footprint (none) -> bus_beaglebone:Pin_Header_Straight_1x03
- J2: footprint (none) -> bus_beaglebone:Pin_Header_Straight_2x02
- N1, N2: footprint (none) -> bus_beaglebone:5MM_TERMINAL_BLOCK_2_POS
- N10: footprint (none) -> bus_beaglebone:Pin_Header_Straight_2x23
- N3, N9: footprint (none) -> bus_beaglebone:Pin_Header_Straight_2x05_Shrouded
- N4, N5: footprint (none) -> bus_beaglebone:Pin_Header_Straight_1x06
- N6: footprint (none) -> bus_beaglebone:OKI_DC_TO_DC_CONNECTOR
- N7: footprint (none) -> bus_beaglebone:Pin_Header_Straight_2x03
- N8: footprint (none) -> bus_beaglebone:Pin_Header_Straight_1x04
- Q1: footprint (none) -> bus_beaglebone:TO-220_FET-GDS_Horizontal_LargePads
- R3, R4, R5, R6: footprint (none) -> bus_beaglebone:Resistor_Horizontal__400
- SW1: footprint (none) -> bus_beaglebone:Button_6.5MM
- U1: footprint (none) -> bus_beaglebone:DIP-14__300
- U2: footprint (none) -> bus_beaglebone:DIP-8__300
- U3: footprint (none) -> bus_beaglebone:DIP-40__600
- X1: footprint (none) -> bus_beaglebone:Crystal_HC49-U_Vertical
- X2: footprint (none) -> bus_beaglebone:OSHW_LOGO_250mil
Connections:
- net +5V: now also N10.5 (VDD_5V), N10.6 (VDD_5V), R1.1, R1.1, R1.1, R1.1; no longer N10.11 (GPIO30_UART4_RX), N10.12 (GPIO60)
- net GND: now also N10.1 (DGND), N10.2 (DGND), N10.43 (DGND), N10.44 (DGND), N10.45 (DGND), N10.46 (DGND), R8.1, R8.1, R8.1, R8.1; no longer N10.7 (SYS_5V), N10.8 (SYS_5V), U2.8 (STBY)
- net RXD1: now also U2.4 (RXD); no longer U2.1 (TXD)
- net SCK: now also N9.6 (~NRST)
- net TXD0: now also U1.9, R2.2
- net TXD1: now also U2.1 (TXD); no longer U2.4 (RXD)
- net at U3.20 (PD6/OC2B): now also U2.8 (STBY)
- net at C8.2, U1.11: no longer N9.6 (~NRST)
- net at N5.5 (RXD), N8.2 (TXD), U1.5: now also N10.21 (GPIO3_UART2_TX), R1.5, R8.5; no longer N10.27 (GPIO125)
- net at N4.4 (TXD), U1.4: now also R1.3
- net at N4.5 (RXD): now also R2.1, R8.2; no longer U1.9
- net at N4.6 (~RTS), U1.2: now also R1.2
- net at U1.8: now also R7.2
- net at N8.4 (~RESET), U1.12: now also N10.31 (GPIO110_SPI1_SCLK), R1.4, R8.4; no longer N10.37 (AIN2)
- net at N8.3 (RXD): now also N10.22 (GPIO2_UART2_RX), R7.1, R8.3; no longer N10.28 (GPIO113_SPI1_CS0)
- no-connect marks 60 -> 69
Other:
- moved on the sheet: H1, H2, H3, H4, N10

Commit message: Checked in Rev. B
Parts:
- N6: value OKI-77SR-5/1.5-W36-C -> OKI-78SR-5/1.5-W36-C
- R1: value 22K -> 22K_SIP5
- R8: value 33K -> 33K_SIP5
Other:
- moved on the sheet: R1A, R1B, R1D, R8A, R8D
Changed lines of the file:
@@
 LIBS:valves
 LIBS:bus_beaglebone-cache
-EELAYER 24 0
+EELAYER 25 0
 EELAYER END
 $Descr A 11000 8500
@@
 L GND #PWR09
 U 1 1 53E41588
-P 8550 6500
-F 0 "#PWR09" H 8550 6500 30  0001 C CNN
-F 1 "GND" H 8550 6430 30  0001 C CNN
-F 2 "" H 8550 6500 60  0000 C CNN
-F 3 "" H 8550 6500 60  0000 C CNN
-	1    8550 6500
+P 8500 6500
+F 0 "#PWR09" H 8500 6500 30  0001 C CNN
+F 1 "GND" H 8500 6430 30  0001 C CNN
+F 2 "" H 8500 6500 60  0000 C CNN
+F 3 "" H 8500 6500 60  0000 C CNN
+	1    8500 6500
 	1    0    0    -1
 $EndComp
@@
 P 4150 7200
 F 0 "N6" H 4050 7400 50  0000 C CNN
-F 1 "OKI-77SR-5/1.5-W36-C" H 4150 7000 50  0000 C CNN
+F 1 "OKI-78SR-5/1.5-W36-C" H 4150 7000 50  0000 C CNN
 F 2 "bus_beaglebone:OKI_DC_TO_DC_CONNECTOR" H 4150 7200 60  0001 C CNN
 F 3 "" H 4150 7200 60  0000 C CNN
@@
 L +5V #PWR020
 U 1 1 53E62621
-P 2400 2500
-F 0 "#PWR020" H 2400 2590 20  0001 C CNN
-F 1 "+5V" H 2390 2615 50  0000 C CNN
-F 2 "" H 2400 2500 60  0000 C CNN
-F 3 "" H 2400 2500 60  0000 C CNN
-	1    2400 2500
+P 2300 2500
+F 0 "#PWR020" H 2300 2590 20  0001 C CNN
+F 1 "+5V" H 2290 2615 50  0000 C CNN
+F 2 "" H 2300 2500 60  0000 C CNN
+F 3 "" H 2300 2500 60  0000 C CNN
+	1    2300 2500
 	1    0    0    -1
 $EndComp
@@
 L +5V #PWR021
 U 1 1 53E64BEC
-P 1900 2500
-F 0 "#PWR021" H 1900 2590 20  0001 C CNN
-F 1 "+5V" H 1890 2615 50  0000 C CNN
-F 2 "" H 1900 2500 60  0000 C CNN
-F 3 "" H 1900 2500 60  0000 C CNN
-	1    1900 2500
+P 1800 2500
+F 0 "#PWR021" H 1800 2590 20  0001 C CNN
+F 1 "+5V" H 1790 2615 50  0000 C CNN
+F 2 "" H 1800 2500 60  0000 C CNN
+F 3 "" H 1800 2500 60  0000 C CNN
+	1    1800 2500
 	1    0    0    -1
 $EndComp
@@
 L GND #PWR022
 U 1 1 53E6A5C3
-P 4400 3800
-F 0 "#PWR022" H 4400 3800 30  0001 C CNN
-F 1 "GND" H 4400 3730 30  0001 C CNN
-F 2 "" H 4400 3800 60  0000 C CNN
-F 3 "" H 4400 3800 60  0000 C CNN
-	1    4400 3800
+P 3800 3800
+F 0 "#PWR022" H 3800 3800 30  0001 C CNN
+F 1 "GND" H 3800 3730 30  0001 C CNN
+F 2 "" H 3800 3800 60  0000 C CNN
+F 3 "" H 3800 3800 60  0000 C CNN
+	1    3800 3800
 	1    0    0    -1
 $EndComp
@@
 U 1 1 53E7BE34
 P 7900 6250
-F 0 "N8" H 7900 6550 60  0000 C CNN
+F 0 "N8" H 7700 6550 60  0000 C CNN
 F 1 "SERIAL_CONNECTOR" H 7900 5925 50  0000 C CNN
 F 2 "bus_beaglebone:Pin_Header_Straight_1x04" H 7900 6250 60  0001 C CNN
@@
 	2800 2800 3000 2800
 Wire Wire Line
-	1300 3100 1900 3100
-Wire Wire Line
-	8650 4300 9300 4300
+	1300 3100 1800 3100
+Wire Wire Line
+	8600 4300 9300 4300
 Wire Wire Line
 	7500 5500 7500 5700
@@
 	2200 6400 2200 6600
 Wire Wire Line
-	3400 6600 2200 6600
-Wire Wire Line
-	3400 6000 3400 6600
+	2200 6600 3400 6600
+Wire Wire Line
+	3400 6600 3400 6000
 Wire Wire Line
 	3300 6300 3400 6300
@@
 	1600 5500 1600 5700
 Wire Wire Line
-	8550 4200 9300 4200
+	8500 4200 9300 4200
 Wire Wire Line
 	3500 1500 4300 1500
 Wire Wire Line
-	8650 4300 8650 6200
-Wire Wire Line
-	8650 5600 7500 5600
+	8600 4300 8600 6200
+Wire Wire Line
+	8600 5600 7500 5600
 Connection ~ 7500 5600
 Wire Wire Line
@@
 Wire Wire Line
 	2900 3000 2900 4300
-Connection ~ 2400 3300
-Wire Wire Line
-	2400 2600 2400 2500
+Connection ~ 2300 3300
+Wire Wire Line
+	2300 2600 2300 2500
 Wire Wire Line
 	4100 2200 4100 2900
@@
 	4100 2900 4000 2900
 Wire Wire Line
-	1900 2600 1900 2500
+	1800 2600 1800 2500
 Connection ~ 1700 3100
 Wire Wire Line
 	4400 2600 4400 2300
 Wire Wire Line
-	4400 3000 4400 3300
-Wire Wire Line
-	4400 3800 4400 3700
-Connection ~ 4400 3200
+	3800 3800 3800 3700
 Wire Wire Line
 	6100 5900 6000 5900
@@
 	7700 2400 7200 2400
 Wire Wire Line
-	9000 4900 9000 4800
-Wire Wire Line
-	3900 4500 8550 4500
-Wire Wire Line
-	8550 4200 8550 6300
-Connection ~ 9000 4200
+	8750 4900 8750 4800
+Wire Wire Line
+	3900 4500 8500 4500
+Wire Wire Line
+	8500 4200 8500 6300
+Connection ~ 8750 4200
 Wire Wire Line
 	4800 4100 5600 4100
@@
 Connection ~ 3000 7700
 Wire Wire Line
-	5500 800  5500 1800
-Wire Wire Line
-	1900 800  5500 800
+	5500 1800 5500 800
+Wire Wire Line
+	5500 800  1900 800
 Wire Wire Line
 	1700 1600 2000 1600
@@
 Connection ~ 8400 5200
 Wire Wire Line
-	8550 6300 8300 6300
-Wire Wire Line
-	8650 6200 8300 6200
-Connection ~ 8650 5600
+	8500 6300 8300 6300
+Wire Wire Line
+	8600 6200 8300 6200
+Connection ~ 8600 5600
 Text Label 1150 7100 0    50   ~ 0
 BAT+
@@
 L GND #PWR027
 U 1 1 53E87E15
-P 9000 4900
-F 0 "#PWR027" H 9000 4900 30  0001 C CNN
-F 1 "GND" H 9000 4830 30  0001 C CNN
-F 2 "" H 9000 4900 60  0000 C CNN
-F 3 "" H 9000 4900 60  0000 C CNN
-	1    9000 4900
+P 8750 4900
+F 0 "#PWR027" H 8750 4900 30  0001 C CNN
+F 1 "GND" H 8750 4830 30  0001 C CNN
+F 2 "" H 8750 4900 60  0000 C CNN
+F 3 "" H 8750 4900 60  0000 C CNN
+	1    8750 4900
 	1    0    0    -1
 $EndComp
@@
 L +5V #PWR028
 U 1 1 53E87FB6
-P 9000 3575
-F 0 "#PWR028" H 9000 3665 20  0001 C CNN
-F 1 "+5V" H 8990 3690 50  0000 C CNN
-F 2 "" H 9000 3575 60  0000 C CNN
-F 3 "" H 9000 3575 60  0000 C CNN
-	1    9000 3575
-	1    0    0    -1
-$EndComp
-Wire Wire Line
-	9000 3700 9000 3575
+P 8750 3575
+F 0 "#PWR028" H 8750 3665 20  0001 C CNN
+F 1 "+5V" H 8740 3690 50  0000 C CNN
+F 2 "" H 8750 3575 60  0000 C CNN
+F 3 "" H 8750 3575 60  0000 C CNN
+	1    8750 3575
+	1    0    0    -1
+$EndComp
+Wire Wire Line
+	8750 3700 8750 3575
 NoConn ~ 9300 2400
 NoConn ~ 9300 2500
@@
 NoConn ~ 9300 4600
 Wire Wire Line
-	8550 6500 8550 6400
+	8500 6500 8500 6400
 Wire Wire Line
 	8300 6400 9300 6400
 Connection ~ 5200 3000
 Wire Wire Line
-	9000 4100 9000 4400
-Connection ~ 8550 4500
+	8750 4100 8750 4400
+Connection ~ 8500 4500
 NoConn ~ 9300 5400
 NoConn ~ 9300 5500
@@
 Connection ~ 9200 6500
 Connection ~ 9200 6400
-Connection ~ 8550 6400
+Connection ~ 8500 6400
 Wire Wire Line
 	4700 2300 4700 4900
@@
 	4400 3200 1300 3200
 Wire Wire Line
-	2400 3300 2400 3000
-Wire Wire Line
-	1900 3100 1900 3000
+	2300 3300 2300 3000
+Wire Wire Line
+	1800 3100 1800 3000
 Wire Wire Line
 	7900 3300 7900 3500
@@
 L R_VERT_SIP5 R1
 U 1 1 54308E62
-P 1900 2800
-F 0 "R1" H 1945 2870 50  0000 L CNN
-F 1 "22K" H 1945 2770 50  0000 L CNN
-F 2 "bus_beaglebone:Pin_Header_Straight_1x05" H 1900 2800 50  0001 C CNN
-F 3 "" H 1900 2800 50  0000 C CNN
-	1    1900 2800
+P 1800 2800
+F 0 "R1" H 1845 2870 50  0000 L CNN
+F 1 "22K_SIP5" H 1845 2770 50  0000 L CNN
+F 2 "bus_beaglebone:Pin_Header_Straight_1x05" H 1800 2800 50  0001 C CNN
+F 3 "" H 1800 2800 50  0000 C CNN
+	1    1800 2800
 	1    0    0    -1
 $EndComp
@@
 L R_VERT_SIP5 R1
 U 2 1 54308F11
-P 2400 2800
-F 0 "R1" H 2445 2870 50  0000 L CNN
-F 1 "22K" H 2445 2770 50  0000 L CNN
-F 2 "bus_beaglebone:Pin_Header_Straight_1x05" H 2400 2800 50  0001 C CNN
-F 3 "" H 2400 2800 50  0000 C CNN
-	2    2400 2800
+P 2300 2800
+F 0 "R1" H 2345 2870 50  0000 L CNN
+F 1 "22K_SIP5" H 2345 2770 50  0000 L CNN
+F 2 "bus_beaglebone:Pin_Header_Straight_1x05" H 2300 2800 50  0001 C CNN
+F 3 "" H 2300 2800 50  0000 C CNN
+	2    2300 2800
 	1    0    0    -1
 $EndComp
@@
 P 7900 3100
 F 0 "R1" H 7945 3170 50  0000 L CNN
-F 1 "22K" H 7945 3070 50  0000 L CNN
+F 1 "22K_SIP5" H 7945 3070 50  0000 L CNN
 F 2 "bus_beaglebone:Pin_Header_Straight_1x05" H 7900 3100 50  0001 C CNN
 F 3 "" H 7900 3100 50  0000 C CNN
@@
 L R_VERT_SIP5 R1
 U 4 1 543090B1
-P 9000 3900
-F 0 "R1" H 9045 3970 50  0000 L CNN
-F 1 "22K" H 9045 3870 50  0000 L CNN
-F 2 "bus_beaglebone:Pin_Header_Straight_1x05" H 9000 3900 50  0001 C CNN
-F 3 "" H 9000 3900 50  0000 C CNN
-	4    9000 3900
+P 8750 3900
+F 0 "R1" H 8795 3970 50  0000 L CNN
+F 1 "22K_SIP5" H 8795 3870 50  0000 L CNN
+F 2 "bus_beaglebone:Pin_Header_Straight_1x05" H 8750 3900 50  0001 C CNN
+F 3 "" H 8750 3900 50  0000 C CNN
+	4    8750 3900
 	1    0    0    -1
 $EndComp
@@
 L R_VERT_SIP5_ALT R8
 U 1 1 54309581
-P 4400 3500
-F 0 "R8" H 4445 3570 50  0000 L CNN
-F 1 "33K" H 4445 3470 50  0000 L CNN
-F 2 "bus_beaglebone:Pin_Header_Straight_1x05" H 4400 3500 50  0001 C CNN
-F 3 "" H 4400 3500 50  0000 C CNN
-	1    4400 3500
+P 3800 3500
+F 0 "R8" H 3845 3570 50  0000 L CNN
+F 1 "33K_SIP5" H 3845 3470 50  0000 L CNN
+F 2 "bus_beaglebone:Pin_Header_Straight_1x05" H 3800 3500 50  0001 C CNN
+F 3 "" H 3800 3500 50  0000 C CNN
+	1    3800 3500
 	1    0    0    -1
 $EndComp
@@
 P 7500 5900
 F 0 "R8" H 7545 5970 50  0000 L CNN
-F 1 "33K" H 7545 5870 50  0000 L CNN
+F 1 "33K_SIP5" H 7545 5870 50  0000 L CNN
 F 2 "bus_beaglebone:Pin_Header_Straight_1x05" H 7500 5900 50  0001 C CNN
 F 3 "" H 7500 5900 50  0000 C CNN
@@
 P 7900 3700
 F 0 "R8" H 7945 3770 50  0000 L CNN
-F 1 "33K" H 7945 3670 50  0000 L CNN
+F 1 "33K_SIP5" H 7945 3670 50  0000 L CNN
 F 2 "bus_beaglebone:Pin_Header_Straight_1x05" H 7900 3700 50  0001 C CNN
 F 3 "" H 7900 3700 50  0000 C CNN
@@
 L R_VERT_SIP5_ALT R8
 U 4 1 54309962
-P 9000 4600
-F 0 "R8" H 9045 4670 50  0000 L CNN
-F 1 "33K" H 9045 4570 50  0000 L CNN
-F 2 "bus_beaglebone:Pin_Header_Straight_1x05" H 9000 4600 50  0001 C CNN
-F 3 "" H 9000 4600 50  0000 C CNN
-	4    9000 4600
+P 8750 4600
+F 0 "R8" H 8795 4670 50  0000 L CNN
+F 1 "33K_SIP5" H 8795 4570 50  0000 L CNN
+F 2 "bus_beaglebone:Pin_Header_Straight_1x05" H 8750 4600 50  0001 C CNN
+F 3 "" H 8750 4600 50  0000 C CNN
+	4    8750 4600
 	1    0    0    -1
 $EndComp
@@
 Wire Wire Line
 	2200 5800 2200 6100
+Wire Wire Line
+	3800 3300 3800 3200
+Connection ~ 3800 3200
+Wire Wire Line
+	4400 3000 4400 3200
 $EndSCHEMATC
