File: rev_c/bus_beaglebone.kicad_pcb (KiCad board)
At the start: 2 copper layers, 100 x 50 mm, 46 parts, among them J1 TERMINATE_JUMPER, J2 LED_JUMPER, Q1 FQP47P06, SW1 MJTP1243, U1 74HCT08, U2 MCP2562, U3 ATMEGA324_DIP40, U4 MCP7940, X1 16MHz, X2 OSHW_LOGO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

Commit message: Wrapped up Rev. C.
Parts:
- removed X3: 32.768KHz, bus_beaglebone:RTC_CRYSTAL
- added H5: OSHW_LOGO, bus_beaglebone:OSHW_LOGO_250mil, B.Cu at (141.0, 125.7)
- added N11: KEY, bus_beaglebone:Pin_Header_Straight_1x01, B.Cu at (102.2, 102.9)
- added N12: KEY, bus_beaglebone:Pin_Header_Straight_1x01, B.Cu at (163.2, 102.9)
- added N13: KEY, bus_beaglebone:Pin_Header_Straight_1x01, B.Cu at (134.0, 106.7)
- X2: value OSHW_LOGO -> 32.768KHz; footprint bus_beaglebone:OSHW_LOGO_250mil -> bus_beaglebone:RTC_CRYSTAL; moved to F.Cu
- moved X2 75.8 mm to (125.7, 144.1), turned to 90 degrees
- moved N5 70.0 mm to (191.1, 112.4)
- moved R9 52.6 mm to (109.5, 107.3), turned to 180 degrees
- moved R10 39.1 mm to (122.7, 106.8), turned to 180 degrees
- moved BAT1 30.1 mm to (173.4, 138.4), turned to 180 degrees
- moved R3 10.2 mm to (193.0, 136.5)
- moved U4 7.65 mm to (134.6, 141.6), turned to 270 degrees
- moved C8 3.86 mm to (166.4, 104.8)
- moved N7 3.86 mm to (142.9, 141.0)
- moved C7 3.81 mm to (169.5, 105.4)
- moved U1 2.54 mm to (181.0, 105.4)
- moved N10 2.29 mm to (132.7, 102.9)
- moved R5 1.42 mm to (120.0, 109.9)
- moved R6 1.42 mm to (120.0, 113.0)
- moved D1 1.27 mm to (123.8, 116.2)
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Connections:
- net +5V renamed VCC
- BAT1 pad +: (no net) -> Net-(BAT1-Pad+)
- BAT1 pad -: (no net) -> GND
- N5 pad 1: (no net) -> GND
- N5 pad 4: (no net) -> Net-(N5-Pad4)
- N5 pad 5: (no net) -> Net-(N10-Pad21)
- U1 pad 10: (no net) -> Net-(N5-Pad4)
- U4 pad 1: (no net) -> Net-(U4-Pad1)
- U4 pad 2: (no net) -> Net-(U4-Pad2)
- U4 pad 3: (no net) -> Net-(BAT1-Pad+)
Routing:
- net (no net): track 111.2 -> 0.00 mm, vias 2 -> 0
- net Net-(N10-Pad20): track 0.00 -> 74.3 mm, vias 0 -> 1
- net Net-(BAT1-Pad+): track 0.00 -> 68.0 mm
- net GND: track 325.4 -> 380.3 mm, vias 18 -> 19
- net +3.3V: track 11.6 -> 63.5 mm, vias 0 -> 1
- net Net-(N10-Pad19): track 11.7 -> 50.1 mm
- net Net-(N10-Pad21): track 103.9 -> 86.6 mm
- net Net-(N5-Pad4): track 0.00 -> 14.5 mm
- net /SCK: track 88.7 -> 80.9 mm, vias 1 -> 2
- net Net-(U4-Pad1): track 0.00 -> 6.91 mm
- net /~RESET: track 137.6 -> 143.3 mm
- net Net-(N10-Pad31): track 62.6 -> 68.2 mm, vias 0 -> 1
- net /CANH: track 25.4 -> 21.0 mm
- net Net-(U4-Pad2): track 0.00 -> 4.30 mm
- net Net-(R7-Pad2): track 31.2 -> 26.9 mm
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Other:
- board text added: "(c) Copyright 20014 by Wayne Gramlich"
- board text added: "BUS BEAGLEBONE REV. B 19OCT2014"
- board text added: "OFF"
- board text added: "ON"
- board text added: "PROGRAM"
- board text removed: "1 PROGRAM"
- board text removed: "BUS BEAGLEBONE REV. B 4OCT2014 (c) 2014 GRAMLICH"
- board text removed: "ON/OFF"

Commit message: Wrapped up Rev. C
Other:
- board text added: "BUS BEAGLEBONE REV. C 19OCT2014"
- board text removed: "BUS BEAGLEBONE REV. B 19OCT2014"
