File: rev_c/bus_beaglebone.sch (KiCad schematic (older format))
At the start: 46 parts, among them J1 TERMINATE_JUMPER, J2 LED_JUMPER, Q1 FQP47P06, SW1 MJTP1243, U1 74HCT08, U2 MCP2562, U3 ATMEGA324_DIP40, X1 16MHz, X2 OSHW_LOGO

Commit message: Wrapped up Rev. C.
Parts:
- removed X?: 32.768KHz, bus_beaglebone:Crystal_HC49-U_Vertical, symbol CRYSTAL
- added N11, N12, N13: KEY, bus_beaglebone:Pin_Header_Straight_1x01, symbol KEY
- added X2: 32.768KHz, bus_beaglebone:RTC_CRYSTAL, symbol RTC_CRYSTAL
- BAT1: renamed from BAT?; footprint (none) -> bus_beaglebone:10MM_BATTERY
- U4: renamed from U?; footprint (none) -> bus_beaglebone:DIP-8__300
- gave numbers to parts that had none: 2
- renumbered X2 to H5
Connections:
- net GND: now also N5.1 (GND), N11.1 (GND), N12.1 (GND), N13.1 (GND), X2.3 (GND), X2.4 (GND)
- net at N5.4 (TXD): now also U1.10
- net at N5.5 (RXD): now also N10.21 (GPIO3_UART2_TX), N8.2 (TXD), R1.5, R8.5, U1.5
- net at U4.1 (X1): now also X2.1
- net at U4.2 (X2): now also X2.2
Other:
- note added: "3V Lithium\n>100mAH"
- note removed: "3V Lithium"
- moved on the sheet: BAT1, H1, H2, H3, H4, H5, N5
